File: hardware/schematics/openEMSstim_03.sch (EAGLE design)
At the start: 37 parts

Commit message: new board design V3: not tested yet
Parts:
- added SW1: SW1, alps:SSSS810701
- D1: value 1N4001 -> 1PS70SB10; device semicon-smd-ipc:D-SMB -> nxp_60:1PS70SB10
Connections:
- new net N$64: D1.K, SW1.COM
- net N$11: now also SW1.B; no longer D1.C
Other:
- note added: "Pedro R2 / Dec-2016 - new: diode for reverse batt polarity - new: jumper-pads for diode bypass - new: ON/OFF slide slitch"
Changed lines of the file:
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@@
 <layer number="112" name="tSilk" color="7" fill="1" visible="yes" active="yes"/>
 <layer number="113" name="IDFDebug" color="7" fill="1" visible="yes" active="yes"/>
+<layer number="114" name="FRNTMAAT1" color="7" fill="1" visible="yes" active="yes"/>
+<layer number="115" name="FRNTMAAT2" color="7" fill="1" visible="yes" active="yes"/>
 <layer number="116" name="Patch_BOT" color="9" fill="4" visible="yes" active="yes"/>
+<layer number="117" name="BACKMAAT1" color="7" fill="1" visible="yes" active="yes"/>
 <layer number="118" name="Rect_Pads" color="7" fill="1" visible="no" active="no"/>
+<layer number="119" name="KAP_TEKEN" color="7" fill="1" visible="yes" active="yes"/>
+<layer number="120" name="KAP_MAAT1" color="7" fill="1" visible="yes" active="yes"/>
 <layer number="121" name="_tsilk" color="7" fill="1" visible="yes" active="yes"/>
 <layer number="122" name="_bsilk" color="7" fill="1" visible="yes" active="yes"/>
@@
 <layer number="128" name="_bValues" color="7" fill="1" visible="yes" active="yes"/>
 <layer number="129" name="Mask" color="7" fill="1" visible="yes" active="yes"/>
+<layer number="130" name="SMDSTROOK" color="7" fill="1" visible="yes" active="yes"/>
 <layer number="131" name="tAdjust" color="7" fill="1" visible="yes" active="yes"/>
 <layer number="132" name="bAdjust" color="7" fill="1" visible="yes" active="yes"/>
@@
 <part name="C1" library="SparkFun-Passives" deviceset="CAP" device="0805" value="100nf"/>
 <part name="C3" library="SparkFun-Passives" deviceset="CAP" device="0805" value="100nf"/>
-<part name="D1" library="semicon-smd-ipc" deviceset="D-" device="SMB" value="1N4001"/>
+<part name="D1" library="nxp_60" deviceset="1PS70SB10" device=""/>
+<part name="SW1" library="alps" deviceset="SSSS810701" device="" value="SW1"/>
 </parts>
 <sheets>
@@
 <plain>
 <text x="-347.98" y="177.8" size="1.778" layer="91">DO not use D10</text>
+<text x="-508" y="228.6" size="1.778" layer="91">Pedro R2 / Dec-2016
+- new: diode for reverse batt polarity
+- new: jumper-pads for diode bypass
+- new: ON/OFF slide slitch</text>
 </plain>
 <instances>
@@
 <instance part="C1" gate="G$1" x="-416.56" y="106.68"/>
 <instance part="C3" gate="G$1" x="-177.8" y="91.44"/>
-<instance part="D1" gate="G$1" x="-414.02" y="213.36"/>
+<instance part="D1" gate="G$1" x="-411.48" y="213.36"/>
+<instance part="SW1" gate="G$1" x="-396.24" y="215.9"/>
 </instances>
 <busses>
@@
 <segment>
 <pinref part="MODUL1" gate="G$1" pin="VIN"/>
-<wire x1="-383.54" y1="210.82" x2="-383.54" y2="213.36" width="0.1524" layer="91"/>
-<pinref part="D1" gate="G$1" pin="C"/>
-<wire x1="-411.48" y1="213.36" x2="-383.54" y2="213.36" width="0.1524" layer="91"/>
+<pinref part="SW1" gate="G$1" pin="B"/>
+<wire x1="-396.24" y1="215.9" x2="-383.54" y2="215.9" width="0.1524" layer="91"/>
+<wire x1="-383.54" y1="215.9" x2="-383.54" y2="210.82" width="0.1524" layer="91"/>
 </segment>
 </net>
@@
 <pinref part="JP1" gate="G$1" pin="1"/>
 <pinref part="D1" gate="G$1" pin="A"/>
-<wire x1="-429.26" y1="213.36" x2="-416.56" y2="213.36" width="0.1524" layer="91"/>
+<wire x1="-429.26" y1="213.36" x2="-414.02" y2="213.36" width="0.1524" layer="91"/>
+</segment>
+</net>
+<net name="N$64" class="0">
+<segment>
+<pinref part="D1" gate="G$1" pin="K"/>
+<pinref part="SW1" gate="G$1" pin="COM"/>
+<wire x1="-408.94" y1="213.36" x2="-398.78" y2="213.36" width="0.1524" layer="91"/>
+<wire x1="-398.78" y1="213.36" x2="-398.78" y2="218.44" width="0.1524" layer="91"/>
 </segment>
 </net>
@@
 </schematic>
 </drawing>
+<compatibility>
+<note version="6.3" minversion="6.2.2" severity="warning">
+Since Version 6.2.2 text objects can contain more than one line,
+which will not be processed correctly with this version.
+</note>
+</compatibility>
 </eagle>
